Commit message: replaced race car model

File: models/vehicles/racecar/racecar.urdf (robot description, URDF)
Before this commit: robot racecar, 13 links, 12 joints
Links:
- removed link base_link
- removed link chassis_inertia
- added link diff2_ring, mass 0.0637; collision cylinder length=0.01 radius=0.025; visual mesh filename=differential/diff_carrier.stl scale=0.001 0.001 0.001
- added link diff2_sideA, mass 0.056; collision cylinder length=0.01 radius=0.015; visual mesh filename=differential/diff_side.stl scale=0.001 0.001 0.001
- added link diff2_sideB, mass 0.056; collision cylinder length=0.01 radius=0.015; visual mesh filename=differential/diff_side.stl scale=0.001 0.001 0.001
- added link diff2_spiderA, mass 0.056; collision cylinder length=0.01 radius=0.015; visual mesh filename=differential/diff_spider.stl scale=0.001 0.001 0.001
- added link diff2_spiderB, mass 0.056; collision cylinder length=0.01 radius=0.015; visual mesh filename=differential/diff_spider.stl scale=0.001 0.001 0.001
- added link diff_ring, mass 0.0637; collision cylinder length=0.01 radius=0.025; visual mesh filename=differential/diff_carrier.stl scale=0.001 0.001 0.001
- added link diff_sideA, mass 0.056; collision cylinder length=0.01 radius=0.015; visual mesh filename=differential/diff_side.stl scale=0.001 0.001 0.001
- added link diff_sideB, mass 0.056; collision cylinder length=0.01 radius=0.015; visual mesh filename=differential/diff_side.stl scale=0.001 0.001 0.001
- added link diff_spiderA, mass 0.056; collision cylinder length=0.01 radius=0.015; visual mesh filename=differential/diff_spider.stl scale=0.001 0.001 0.001
- added link diff_spiderB, mass 0.056; collision cylinder length=0.01 radius=0.015; visual mesh filename=differential/diff_spider.stl scale=0.001 0.001 0.001
- link camera_link: mass 1e-5 -> 0.01
- link chassis: mass .1 -> 4.0; geometry collision mesh filename=meshes/chassis_differential.STL scale=1 1 1 1; visual mesh filename=meshes/chassis_differential.STL scale=1 1 1 1
- link zed_camera_link: mass 1e-5 -> 0.1
- link zed_camera_right_link: mass 1e-5 -> 0.01
Joints:
- removed joint base_link_joint
- removed joint chassis_inertia_joint
- added joint diff2_ring_chassis: type continuous, parent chassis, child diff2_ring, origin xyz=0.32 0.0 0.0 rpy=0 0 0, axis 0 1 0
- added joint diff2_sideA_ring: type continuous, parent diff2_ring, child diff2_sideA, origin xyz=0.0 0.0 0.0 rpy=0 0 0, axis 0 1 0
- added joint diff2_sideB_ring: type continuous, parent diff2_ring, child diff2_sideB, origin xyz=0.0 0.0 0.0 rpy=0 0 0, axis 0 1 0
- added joint diff2_spiderA_ring: type continuous, parent diff2_ring, child diff2_spiderA, origin xyz=0.0 0.0 0.0 rpy=0 0 1.570795, axis 0 1 0
- added joint diff2_spiderB_ring: type continuous, parent diff2_ring, child diff2_spiderB, origin xyz=0.0 0.0 0.0 rpy=0 0 -1.570795, axis 0 1 0
- added joint diff_ring_chassis: type continuous, parent chassis, child diff_ring, origin xyz=0.0 0.0 0. rpy=0 0 0, axis 0 1 0
- added joint diff_sideA_ring: type continuous, parent diff_ring, child diff_sideA, origin xyz=0.0 0.0 0.0 rpy=0 0 0, axis 0 1 0
- added joint diff_sideB_ring: type continuous, parent diff_ring, child diff_sideB, origin xyz=0.0 0.0 0.0 rpy=0 0 0, axis 0 1 0
- added joint diff_spiderA_ring: type continuous, parent diff_ring, child diff_spiderA, origin xyz=0.0 0.0 0.0 rpy=0 0 1.570795, axis 0 1 0
- added joint diff_spiderB_ring: type continuous, parent diff_ring, child diff_spiderB, origin xyz=0.0 0.0 0.0 rpy=0 0 -1.570795, axis 0 1 0
- joint left_rear_wheel_joint: axis 0 0 -1 -> (none); limit effort=10 velocity=100 -> (none); parent chassis -> diff_sideA; type continuous -> fixed
- joint right_rear_wheel_joint: axis 0 0 -1 -> (none); limit effort=10 velocity=100 -> (none); parent chassis -> diff_sideB; type continuous -> fixed

Commit message: - added support for any number of agents - refactored world.py

File: models/vehicles/racecar/racecar.urdf (robot description, URDF)
Before this commit: robot racecar, 21 links, 20 joints
Links:
- link diff_ring: geometry collision cylinder length=0.01 radius=0.025
- link diff_sideA: geometry collision cylinder length=0.01 radius=0.015
- link diff_spiderA: geometry collision cylinder length=0.01 radius=0.015
- link diff_spiderB: geometry collision cylinder length=0.01 radius=0.015
- link left_steering_hinge: geometry 
- link right_steering_hinge: geometry 
